Commit message: last changes repo will be deleted in next clean

File: urdf/ebamk1a.urdf (robot description, URDF)
Before this commit: robot ebamk1, 4 links, 3 joints
Links:
- added link link_4; visual box size=0.01 0.01 0.005
- added link link_5; visual box size=0.01 0.05 0.005
- link base_link: geometry visual cylinder length=0.032 radius=0.035
- link link_1: geometry visual box size=0.01 0.034 0.034
- link link_2: geometry visual box size=0.01 0.01 0.08
Joints:
- added joint joint_4: type revolute, parent link_3, child link_4, origin xyz=0 0.085 0 rpy=0 0 0, axis 1 0 0, limit lower=-0.7854 upper=1.2217 effort=0 velocity=0
- added joint joint_5: type fixed, parent link_4, child link_5, origin xyz=0 0.01 0 rpy=0 0 0, axis 1 0 0
- joint joint_1: origin xyz=0 0 0.05215 rpy=0 0 0 -> xyz=0 0 0.049 rpy=0 0 0
- joint joint_2: origin xyz=0 0 0.01515 rpy=0 0 0 -> xyz=0 0 0.017 rpy=0 0 0
- joint joint_3: origin xyz=0 0 0.095 rpy=0 0 0 -> xyz=0 0 0.08 rpy=0 0 0

File: urdf/ebamk1b.urdf (robot description, URDF)
Before this commit: robot siBOT, 4 links, 3 joints
Links:
- link base_link: geometry visual cylinder length=0.032 radius=0.035
- link link_1: geometry visual box size=0.01 0.034 0.034
- link link_2: geometry visual box size=0.01 0.01 0.08
- link link_3: geometry visual box size=0.0075 0.127 0.01
Joints:
- joint joint_1: origin xyz=0 0 0.05 rpy=0 0 0 -> xyz=0 0 0.049 rpy=0 0 0
- joint joint_2: axis 0 0 1 -> 1 0 0; origin xyz=0 -0.005 0.035 rpy=1.578 0 0 -> xyz=0 0 0.017 rpy=0 0 0
- joint joint_3: axis 0 0 1 -> 1 0 0; origin xyz=-0.021 0.133 -0.0105 rpy=0 0 0 -> xyz=0 0 0.08 rpy=0 0 0
